Commit message: adaptation for emrox integration worked (to check if still works with futama2 project alone)

File: futama2_robot/futama2_description/urdf/futama2.xacro (robot description, xacro)
@@ -1,2 +1,3 @@
+<?xml version="1.0"?>
 <robot xmlns:xacro="http://www.ros.org/wiki/xacro" name="futama2">
   <link name="futama2_base_link">
@@ -24,5 +25,5 @@
   <link name="realsense_tpu_link">
     <inertial>
-      <origin xyz="0.032157 0.00051011 -0.0001135" rpy="0 0 0" />
+      <origin xyz="0.032157 0.00051011 -0.0001135" rpy="0 0 0"/>
       <mass value="0.2645" />
       <inertia ixx="8.7232E-05" ixy="-1.7837E-06" ixz="3.0021E-09" iyy="0.00010899" iyz="-1.976E-08" izz="0.00014445" />

Commit message: move_group switch successful + change in rotation center link to fit link

File: futama2_robot/futama2_description/urdf/futama2.xacro (robot description, xacro)
@@ -100,5 +100,5 @@
     <child link="camera2_link" />
   </joint>
-  <link name="rotation_center_link">
+  <link name="fit_link">
       <inertial>
       <mass value="0.01"/>
@@ -106,8 +106,8 @@
     </inertial>
   </link>
-  <joint name="rotation_center_joint" type="fixed">
-    <origin xyz="0.291129 0.0 0.3105" rpy="0 0 0" />
+  <joint name="fit_joint" type="fixed">
+    <origin xyz="0.08 0.0 0.48" rpy="0 0 0" />
     <parent link="futama2_base_link"/>
-    <child link="rotation_center_link" />
+    <child link="fit_link" />
   </joint>
   <link name="led_back_up_left_link"/>

Commit message: addressed futama2_description package properly for the meshes (helps for Gazebo too)

File: futama2_robot/futama2_description/urdf/futama2.xacro (robot description, xacro)
@@ -10,5 +10,5 @@
       <origin xyz="0 0 0" rpy="0 0 0" />
       <geometry>
-        <mesh filename="package://futama2_description/meshes/visual/base_link.STL" />
+        <mesh filename="$(find futama2_description)/meshes/visual/base_link.STL" />
       </geometry>
       <material name="">
@@ -19,5 +19,5 @@
       <origin xyz="0 0 0" rpy="0 0 0" />
       <geometry>
-        <mesh filename="package://futama2_description/meshes/collision/base_link.STL" />
+        <mesh filename="$(find futama2_description)/meshes/collision/base_link.STL" />
       </geometry>
     </collision>
@@ -32,5 +32,5 @@
       <origin xyz="0 0 0" rpy="0 0 0" />
       <geometry>
-        <mesh filename="package://futama2_description/meshes/visual/realsense_tpu_link.STL" />
+        <mesh filename="$(find futama2_description)/meshes/visual/realsense_tpu_link.STL" />
       </geometry>
       <material name="">
@@ -41,5 +41,5 @@
       <origin xyz="0 0 0" rpy="0 0 0" />
       <geometry>
-        <mesh filename="package://futama2_description/meshes/collision/realsense_tpu_link.STL" />
+        <mesh filename="$(find futama2_description)/meshes/collision/realsense_tpu_link.STL" />
       </geometry>
     </collision>

Commit message: refixed the package source, no usedful to do $ find package. futama working again

File: futama2_robot/futama2_description/urdf/futama2.xacro (robot description, xacro)
@@ -10,5 +10,5 @@
       <origin xyz="0 0 0" rpy="0 0 0" />
       <geometry>
-        <mesh filename="$(find futama2_description)/meshes/visual/base_link.STL" />
+        <mesh filename="package://futama2_description/meshes/visual/base_link.STL" />
       </geometry>
       <material name="">
@@ -19,5 +19,5 @@
       <origin xyz="0 0 0" rpy="0 0 0" />
       <geometry>
-        <mesh filename="$(find futama2_description)/meshes/collision/base_link.STL" />
+        <mesh filename="package://futama2_description/meshes/collision/base_link.STL" />
       </geometry>
     </collision>
@@ -32,5 +32,5 @@
       <origin xyz="0 0 0" rpy="0 0 0" />
       <geometry>
-        <mesh filename="$(find futama2_description)/meshes/visual/realsense_tpu_link.STL" />
+        <mesh filename="package://futama2_description/meshes/visual/realsense_tpu_link.STL" />
       </geometry>
       <material name="">
@@ -41,5 +41,5 @@
       <origin xyz="0 0 0" rpy="0 0 0" />
       <geometry>
-        <mesh filename="$(find futama2_description)/meshes/collision/realsense_tpu_link.STL" />
+        <mesh filename="package://futama2_description/meshes/collision/realsense_tpu_link.STL" />
       </geometry>
     </collision>

Commit message: refactor

File: futama2_robot/futama2_description/urdf/futama2.xacro (robot description, xacro)
@@ -67,15 +67,4 @@
     <child link="realsense_front_link" />
   </joint>
-  <link name="camera_link">
-      <inertial>
-      <mass value="0.01"/>
-      <inertia ixx="0.01" ixy="0.0" ixz="0.0" iyx="0.0" iyy="0.01" iyz="0.0" izx="0.0" izy="0.0" izz="0.01"/>
-    </inertial>
-  </link>
-  <joint name="camera_joint" type="fixed">
-    <origin xyz="0.04 0 0" rpy="0 0 0" />
-    <parent link="realsense_center_link"/>
-    <child link="camera_link" />
-  </joint>
   <link name="camera1_link">
       <inertial>
@@ -85,5 +74,5 @@
   </link>
   <joint name="camera1_joint" type="fixed">
-    <origin xyz="0 0 0.02" rpy="0 -1.5708 1.5708" />
+    <origin xyz="0.04 0 0" rpy="0 0 0" />
     <parent link="realsense_center_link"/>
     <child link="camera1_link" />
@@ -96,7 +85,18 @@
   </link>
   <joint name="camera2_joint" type="fixed">
+    <origin xyz="0 0 0.02" rpy="0 -1.5708 1.5708" />
+    <parent link="realsense_center_link"/>
+    <child link="camera2_link" />
+  </joint>
+  <link name="camera3_link">
+      <inertial>
+      <mass value="0.01"/>
+      <inertia ixx="0.01" ixy="0.0" ixz="0.0" iyx="0.0" iyy="0.01" iyz="0.0" izx="0.0" izy="0.0" izz="0.01"/>
+    </inertial>
+  </link>
+  <joint name="camera3_joint" type="fixed">
     <origin xyz="0 0 -0.02" rpy="0 1.5708 1.5708" />
     <parent link="realsense_center_link"/>
-    <child link="camera2_link" />
+    <child link="camera3_link" />
   </joint>
   <link name="fit_link">

Commit message: removed unused realsense_front_link

File: futama2_robot/futama2_description/urdf/futama2.xacro (robot description, xacro)
@@ -55,15 +55,4 @@
     <parent link="futama2_base_link"/>
     <child link="realsense_center_link" />
-  </joint>
-  <link name="realsense_front_link">
-      <inertial>
-      <mass value="0.01"/>
-      <inertia ixx="0.01" ixy="0.0" ixz="0.0" iyx="0.0" iyy="0.01" iyz="0.0" izx="0.0" izy="0.0" izz="0.01"/>
-    </inertial>
-  </link>
-  <joint name="realsense_front_joint" type="fixed">
-    <origin xyz="0.043 0 0" rpy="0 0 0" />
-    <parent link="realsense_center_link"/>
-    <child link="realsense_front_link" />
   </joint>
   <link name="camera1_link">
